Commit message: .

File: app_ws/src/btkamr_description/urdf/main.urdf.xacro (robot description, xacro)
@@ -22,5 +22,4 @@
     <!-- Dosyaları Dahil Etme -->
     <xacro:include filename="./wheels.urdf.xacro" />
-    <xacro:include filename="./g_plugins.xacro" />
     <!-- Base Link -->
     <link name="base_footprint"/>
@@ -48,8 +47,12 @@
         </inertial>
         <visual>
-            <geometry><box size="${chasis_len_x} ${chasis_len_y} ${chasis_len_z}"/></geometry>
+            <geometry>
+                <box size="${chasis_len_x} ${chasis_len_y} ${chasis_len_z}"/>
+            </geometry>
         </visual>
         <collision>
-            <geometry><box size="${chasis_len_x} ${chasis_len_y} ${chasis_len_z}"/></geometry>
+            <geometry>
+                <box size="${chasis_len_x} ${chasis_len_y} ${chasis_len_z}"/>
+            </geometry>
         </collision>
     </link>

Commit message: .

File: app_ws/src/btkamr_description/urdf/main.urdf.xacro (robot description, xacro)
@@ -22,4 +22,5 @@
     <!-- Dosyaları Dahil Etme -->
     <xacro:include filename="./wheels.urdf.xacro" />
+    <xacro:include filename="./g_plugins.urdf.xacro" />
     <!-- Base Link -->
     <link name="base_footprint"/>
@@ -47,12 +48,8 @@
         </inertial>
         <visual>
-            <geometry>
-                <box size="${chasis_len_x} ${chasis_len_y} ${chasis_len_z}"/>
-            </geometry>
+            <geometry><box size="${chasis_len_x} ${chasis_len_y} ${chasis_len_z}"/></geometry>
         </visual>
         <collision>
-            <geometry>
-                <box size="${chasis_len_x} ${chasis_len_y} ${chasis_len_z}"/>
-            </geometry>
+            <geometry><box size="${chasis_len_x} ${chasis_len_y} ${chasis_len_z}"/></geometry>
         </collision>
     </link>

File: app_ws/src/btkamr_description/urdf/wheels.urdf.xacro (robot description, xacro)
@@ -35,4 +35,5 @@
                     <cylinder radius="${wh_radius}" length="${wh_thick}"/>
                 </geometry>
+                <material name="gray"/>
             </visual>
             <collision>
@@ -76,4 +77,5 @@
                     <sphere radius="${cwh_radius}"/>
                 </geometry>
+                <material name="gray"/>
             </visual>
             <!-- Çarpışma ve sürtünme ayarları -->

Commit message: .

File: app_ws/src/btkamr_description/urdf/main.urdf.xacro (robot description, xacro)
@@ -14,4 +14,7 @@
         <color rgba="0.7 0.7 0.7 1"/>
     </material>
+    <material name="black">
+        <color rgba="0 0 0 1"/>
+    </material>
     <!-- Şase Nitelikleri -->
     <xacro:property name="chasis_len_x" value="0.6"/>
@@ -23,4 +26,5 @@
     <xacro:include filename="./wheels.urdf.xacro" />
     <xacro:include filename="./g_plugins.urdf.xacro" />
+    <xacro:include filename="./sensor_extensions.urdf.xacro" />
     <!-- Base Link -->
     <link name="base_footprint"/>
